File: bomba-robotabor.kicad_pcb (KiCad board)
At the start: 2 copper layers, 103.6 x 61.2 mm, 52 parts, among them U1 74HC03, U2 74HCT08, U3 L4904

Commit message: board shrunk to 10*10 , all pads now round
Parts:
- removed the   at (129.5, 59.7)
- removed the   at (162.6, 48.3)
- removed the   at (138.4, 59.7)
- removed the   at (181.6, 57.1)
- removed the   at (129.5, 57.1)
- removed the   at (116.8, 59.7)
- removed the   at (116.8, 57.1)
- removed the   at (116.8, 69.8)
- removed the   at (167.6, 52.1)
- removed the   at (157.5, 82.5)
- removed the   at (116.8, 72.4)
- removed the   at (160.0, 82.5)
- removed the   at (160.0, 48.3)
- removed the   at (138.4, 57.1)
- removed the   at (163.8, 67.3)
- added  : PinSocket_1x02_P2.54mm_Vertical, Connector_PinSocket_2.54mm:PinSocket_1x02_P2.54mm_Vertical, F.Cu at (159.8, 48.3)
- added  : PinSocket_1x01_P2.54mm_Vertical, Connector_PinSocket_2.54mm:PinSocket_1x01_P2.54mm_Vertical, F.Cu at (182.1, 57.1)
- added  : PinSocket_1x02_P2.54mm_Vertical, Connector_PinSocket_2.54mm:PinSocket_1x02_P2.54mm_Vertical, F.Cu at (130.0, 57.1)
- added  : PinSocket_1x02_P2.54mm_Vertical, Connector_PinSocket_2.54mm:PinSocket_1x02_P2.54mm_Vertical, F.Cu at (116.4, 56.9)
- added  : PinSocket_1x01_P2.54mm_Vertical, Connector_PinSocket_2.54mm:PinSocket_1x01_P2.54mm_Vertical, F.Cu at (168.1, 52.1)
- added  : PinSocket_1x02_P2.54mm_Vertical, Connector_PinSocket_2.54mm:PinSocket_1x02_P2.54mm_Vertical, F.Cu at (136.9, 57.2)
- added  : PinSocket_1x02_P2.54mm_Vertical, Connector_PinSocket_2.54mm:PinSocket_1x02_P2.54mm_Vertical, F.Cu at (116.4, 69.9)
-  : value PinSocket_1x01_P2.54mm_Vertical -> PinSocket_1x03_P2.54mm_Vertical; footprint Connector_PinSocket_2.54mm:PinSocket_1x01_P2.54mm_Vertical -> Connector_PinSocket_2.54mm:PinSocket_1x03_P2.54mm_Vertical
-  : value PinSocket_1x01_P2.54mm_Vertical -> PinSocket_1x02_P2.54mm_Vertical; footprint Connector_PinSocket_2.54mm:PinSocket_1x01_P2.54mm_Vertical -> Connector_PinSocket_2.54mm:PinSocket_1x02_P2.54mm_Vertical
- moved RESET 5.75 mm to (203.9, 89.1), turned to 180 degrees
- moved R (PIEZO) 2.54 mm to (210.3, 76.5)
- moved R (LED) 2.29 mm to (193.8, 91.4)
- moved   1.55 mm to (162.6, 84.1), turned to -90 degrees
- moved   1.52 mm to (162.3, 64.8)
- moved   0.76 mm to (119.6, 77.5)
- moved   0.76 mm to (165.6, 57.1)
- moved   0.76 mm to (165.6, 61.0)
- moved REF** 0.53 mm to (179.6, 64.8)
- moved   0.51 mm to (140.5, 57.1)
- moved   0.51 mm to (136.1, 77.5)
- moved   0.51 mm to (130.0, 64.8)
- moved   0.51 mm to (130.0, 72.4)
- moved   0.51 mm to (154.2, 57.1)
- moved   0.51 mm to (137.7, 52.1)
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Routing:
- net (no net): track 825.4 -> 821.1 mm
Other:
- board size 103.6 x 61.2 mm -> 99.6 x 61.2 mm
- board text removed: "BASIC"
