File: bomba-robotabor.kicad_sch (KiCad schematic)
At the start: 10 parts, among them U1 74HC03, U2 74HCT08, U3 L4904

Commit message: part list added, bunch of junk
Parts:
- R1, R4, R5, R6: value R -> 4.7kR
- R2, R3, R7: value R -> 1kR
- U1, U2: LCSC (none) -> C352835
- U3: LCSC (none) -> C99439
Changed lines of the file:
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@@
+      (effects (font (size 1.27 1.27)) hide)
+    )
+    (property "LCSC" "C99439" (id 4) (at 151.13 85.09 0)
       (effects (font (size 1.27 1.27)) hide)
     )
@@
     (property "Package" "DIP254P762X508-14" (id 5) (at 41.91 91.44 0)
       (effects (font (size 1.27 1.27)) (justify left bottom) hide)
+    )
+    (property "LCSC" "C352835" (id 6) (at 41.91 91.44 0)
+      (effects (font (size 1.27 1.27)) hide)
     )
     (pin "1")
@@
       (effects (font (size 1.27 1.27)) (justify left bottom) hide)
     )
+    (property "LCSC" "C352835" (id 6) (at 96.52 91.44 0)
+      (effects (font (size 1.27 1.27)) hide)
+    )
     (pin "1")
     (pin "10")
@@
     (in_bom yes) (on_board yes)
     (property "Reference" "R5" (id 0) (at 133.35 76.0222 90))
-    (property "Value" "R" (id 1) (at 133.35 78.3336 90))
+    (property "Value" "4.7kR" (id 1) (at 133.35 78.3336 90))
     (property "Footprint" "Resistor_THT:R_Axial_DIN0207_L6.3mm_D2.5mm_P10.16mm_Horizontal" (id 2) (at 133.35 79.502 90)
       (effects (font (size 1.27 1.27)) hide)
@@
       (effects (font (size 1.27 1.27)) (justify left))
     )
-    (property "Value" "R" (id 1) (at 75.438 86.233 0)
+    (property "Value" "1kR" (id 1) (at 75.438 86.233 0)
       (effects (font (size 1.27 1.27)) (justify left))
     )
@@
     (in_bom yes) (on_board yes)
     (property "Reference" "R7" (id 0) (at 124.46 112.8522 90))
-    (property "Value" "R" (id 1) (at 124.46 115.1636 90))
+    (property "Value" "1kR" (id 1) (at 124.46 115.1636 90))
     (property "Footprint" "Resistor_THT:R_Axial_DIN0207_L6.3mm_D2.5mm_P10.16mm_Horizontal" (id 2) (at 124.46 116.332 90)
       (effects (font (size 1.27 1.27)) hide)
@@
     (in_bom yes) (on_board yes)
     (property "Reference" "R1" (id 0) (at 43.18 59.5122 90))
-    (property "Value" "R" (id 1) (at 43.18 61.8236 90))
+    (property "Value" "4.7kR" (id 1) (at 43.18 61.8236 90))
     (property "Footprint" "Resistor_THT:R_Axial_DIN0207_L6.3mm_D2.5mm_P10.16mm_Horizontal" (id 2) (at 43.18 62.992 90)
       (effects (font (size 1.27 1.27)) hide)
@@
     (in_bom yes) (on_board yes)
     (property "Reference" "R4" (id 0) (at 121.92 78.5622 90))
-    (property "Value" "R" (id 1) (at 121.92 80.8736 90))
+    (property "Value" "4.7kR" (id 1) (at 121.92 80.8736 90))
     (property "Footprint" "Resistor_THT:R_Axial_DIN0207_L6.3mm_D2.5mm_P10.16mm_Horizontal" (id 2) (at 121.92 82.042 90)
       (effects (font (size 1.27 1.27)) hide)
@@
     (in_bom yes) (on_board yes)
     (property "Reference" "R3" (id 0) (at 121.92 91.2622 90))
-    (property "Value" "R" (id 1) (at 121.92 93.5736 90))
+    (property "Value" "1kR" (id 1) (at 121.92 93.5736 90))
     (property "Footprint" "Resistor_THT:R_Axial_DIN0207_L6.3mm_D2.5mm_P10.16mm_Horizontal" (id 2) (at 121.92 94.742 90)
       (effects (font (size 1.27 1.27)) hide)
@@
     (in_bom yes) (on_board yes)
     (property "Reference" "R6" (id 0) (at 133.35 86.1822 90))
-    (property "Value" "R" (id 1) (at 133.35 88.4936 90))
+    (property "Value" "4.7kR" (id 1) (at 133.35 88.4936 90))
     (property "Footprint" "Resistor_THT:R_Axial_DIN0207_L6.3mm_D2.5mm_P10.16mm_Horizontal" (id 2) (at 133.35 89.662 90)
       (effects (font (size 1.27 1.27)) hide)
@@
       (effects (font (size 1.27 1.27)) hide)
     )
-    (property "Value" "+5V" (id 1) (at 42.291 64.1858 0))
+    (property "Value" "+5V" (id 1) (at 44.45 68.58 0))
     (property "Footprint" "" (id 2) (at 41.91 68.58 0)
       (effects (font (size 1.27 1.27)) hide)
@@
     )
     (path "/00000000-0000-0000-0000-0000625f8e3b"
-      (reference "R1") (unit 1) (value "R") (footprint "Resistor_THT:R_Axial_DIN0207_L6.3mm_D2.5mm_P10.16mm_Horizontal")
+      (reference "R1") (unit 1) (value "4.7kR") (footprint "Resistor_THT:R_Axial_DIN0207_L6.3mm_D2.5mm_P10.16mm_Horizontal")
     )
     (path "/00000000-0000-0000-0000-0000625f82fa"
-      (reference "R2") (unit 1) (value "R") (footprint "Resistor_THT:R_Axial_DIN0207_L6.3mm_D2.5mm_P10.16mm_Horizontal")
+      (reference "R2") (unit 1) (value "1kR") (footprint "Resistor_THT:R_Axial_DIN0207_L6.3mm_D2.5mm_P10.16mm_Horizontal")
     )
     (path "/00000000-0000-0000-0000-0000625f9835"
-      (reference "R3") (unit 1) (value "R") (footprint "Resistor_THT:R_Axial_DIN0207_L6.3mm_D2.5mm_P10.16mm_Horizontal")
+      (reference "R3") (unit 1) (value "1kR") (footprint "Resistor_THT:R_Axial_DIN0207_L6.3mm_D2.5mm_P10.16mm_Horizontal")
     )
     (path "/00000000-0000-0000-0000-0000625f965f"
-      (reference "R4") (unit 1) (value "R") (footprint "Resistor_THT:R_Axial_DIN0207_L6.3mm_D2.5mm_P10.16mm_Horizontal")
+      (reference "R4") (unit 1) (value "4.7kR") (footprint "Resistor_THT:R_Axial_DIN0207_L6.3mm_D2.5mm_P10.16mm_Horizontal")
     )
     (path "/00000000-0000-0000-0000-0000625f7399"
-      (reference "R5") (unit 1) (value "R") (footprint "Resistor_THT:R_Axial_DIN0207_L6.3mm_D2.5mm_P10.16mm_Horizontal")
+      (reference "R5") (unit 1) (value "4.7kR") (footprint "Resistor_THT:R_Axial_DIN0207_L6.3mm_D2.5mm_P10.16mm_Horizontal")
     )
     (path "/00000000-0000-0000-0000-0000625f9af4"
-      (reference "R6") (unit 1) (value "R") (footprint "Resistor_THT:R_Axial_DIN0207_L6.3mm_D2.5mm_P10.16mm_Horizontal")
+      (reference "R6") (unit 1) (value "4.7kR") (footprint "Resistor_THT:R_Axial_DIN0207_L6.3mm_D2.5mm_P10.16mm_Horizontal")
     )
     (path "/00000000-0000-0000-0000-0000625f8add"
-      (reference "R7") (unit 1) (value "R") (footprint "Resistor_THT:R_Axial_DIN0207_L6.3mm_D2.5mm_P10.16mm_Horizontal")
+      (reference "R7") (unit 1) (value "1kR") (footprint "Resistor_THT:R_Axial_DIN0207_L6.3mm_D2.5mm_P10.16mm_Horizontal")
     )
     (path "/00000000-0000-0000-0000-0000625d0c38"

Commit message: idk
Parts:
- U1: value 74HC03 -> U1
- U2: value 74HCT08 -> U2
- U3: value L4904 -> U3
Changed lines of the file:
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@@
   )
   (wire (pts (xy 173.99 120.65) (xy 76.2 120.65))
-    (stroke (width 0) (type default) (color 0 0 0 0))
+    (stroke (width 1) (type default) (color 255 0 255 1))
   )
   (wire (pts (xy 171.45 88.9) (xy 171.45 118.11))
@@
   )
   (wire (pts (xy 24.13 64.77) (xy 39.37 64.77))
-    (stroke (width 0) (type default) (color 0 0 0 0))
+    (stroke (width 1) (type default) (color 255 0 0 1))
   )
   (wire (pts (xy 46.99 64.77) (xy 64.77 64.77))
@@
   )
   (wire (pts (xy 76.2 120.65) (xy 76.2 96.52))
-    (stroke (width 0) (type default) (color 0 0 0 0))
+    (stroke (width 1) (type default) (color 255 0 255 1))
   )
   (wire (pts (xy 59.69 81.28) (xy 73.66 81.28))
@@
   )
   (wire (pts (xy 161.29 91.44) (xy 173.99 91.44))
-    (stroke (width 0) (type default) (color 0 0 0 0))
+    (stroke (width 1) (type default) (color 255 0 255 1))
   )
   (wire (pts (xy 173.99 91.44) (xy 173.99 120.65))
-    (stroke (width 0) (type default) (color 0 0 0 0))
+    (stroke (width 1) (type default) (color 255 0 255 1))
   )
   (wire (pts (xy 166.37 99.06) (xy 161.29 99.06))
@@
   )
   (wire (pts (xy 78.74 118.11) (xy 78.74 99.06))
-    (stroke (width 0) (type default) (color 0 0 0 0))
+    (stroke (width 1) (type default) (color 0 0 255 1))
   )
   (wire (pts (xy 73.66 96.52) (xy 73.66 91.44))
-    (stroke (width 0) (type default) (color 0 0 0 0))
+    (stroke (width 1) (type default) (color 0 255 0 1))
   )
   (wire (pts (xy 73.66 91.44) (xy 78.74 91.44))
-    (stroke (width 0) (type default) (color 0 0 0 0))
+    (stroke (width 1) (type default) (color 0 255 0 1))
   )
   (wire (pts (xy 114.3 83.82) (xy 118.11 83.82))
@@
   )
   (wire (pts (xy 73.66 88.9) (xy 78.74 88.9))
-    (stroke (width 0) (type default) (color 0 0 0 0))
+    (stroke (width 1) (type default) (color 255 255 0 1))
   )
   (wire (pts (xy 62.23 62.23) (xy 78.74 62.23))
@@
   )
   (wire (pts (xy 24.13 64.77) (xy 24.13 81.28))
-    (stroke (width 0) (type default) (color 0 0 0 0))
+    (stroke (width 1) (type default) (color 255 0 0 1))
   )
   (wire (pts (xy 120.65 118.11) (xy 78.74 118.11))
-    (stroke (width 0) (type default) (color 0 0 0 0))
+    (stroke (width 1) (type default) (color 0 0 255 1))
   )
   (wire (pts (xy 140.97 91.44) (xy 137.16 91.44))
@@
   )
   (wire (pts (xy 59.69 96.52) (xy 73.66 96.52))
-    (stroke (width 0) (type default) (color 0 0 0 0))
+    (stroke (width 1) (type default) (color 0 255 0 1))
   )
   (wire (pts (xy 140.97 96.52) (xy 125.73 96.52))
@@
       (effects (font (size 1.27 1.27)) hide)
     )
-    (property "Value" "L4904" (id 1) (at 151.13 93.98 0))
+    (property "Value" "U3" (id 1) (at 151.13 93.98 0))
     (property "Footprint" "Package_DIP:DIP-8_W7.62mm" (id 2) (at 151.13 95.25 0)
       (effects (font (size 1.27 1.27)) hide)
@@
       (effects (font (size 1.27 1.27)) (justify left bottom) hide)
     )
-    (property "Value" "74HC03" (id 1) (at 41.91 91.44 0))
+    (property "Value" "U1" (id 1) (at 41.91 91.44 0))
     (property "Footprint" "Package_DIP:DIP-14_W7.62mm" (id 2) (at 41.91 91.44 0)
       (effects (font (size 1.27 1.27)) (justify left bottom) hide)
@@
       (effects (font (size 1.27 1.27)) (justify left bottom) hide)
     )
-    (property "Value" "74HCT08" (id 1) (at 96.52 91.44 0))
+    (property "Value" "U2" (id 1) (at 96.52 91.44 0))
     (property "Footprint" "Package_DIP:DIP-14_W7.62mm" (id 2) (at 96.52 91.44 0)
       (effects (font (size 1.27 1.27)) (justify left bottom) hide)
@@
   (symbol (lib_id "Device:R") (at 73.66 85.09 0) (unit 1)
     (in_bom yes) (on_board yes)
-    (property "Reference" "R2" (id 0) (at 75.438 83.9216 0)
+    (property "Reference" "R2" (id 0) (at 68.58 83.82 0)
       (effects (font (size 1.27 1.27)) (justify left))
     )
-    (property "Value" "1kR" (id 1) (at 75.438 86.233 0)
+    (property "Value" "1kR" (id 1) (at 68.58 86.36 0)
       (effects (font (size 1.27 1.27)) (justify left))
     )
@@
       (effects (font (size 1.27 1.27)) hide)
     )
-    (property "Value" "GND" (id 1) (at 96.647 118.6942 0))
+    (property "Value" "GND" (id 1) (at 100.33 115.57 0))
     (property "Footprint" "" (id 2) (at 96.52 114.3 0)
       (effects (font (size 1.27 1.27)) hide)
@@
     )
     (path "/00000000-0000-0000-0000-0000625d0c38"
-      (reference "U1") (unit 1) (value "74HC03") (footprint "Package_DIP:DIP-14_W7.62mm")
+      (reference "U1") (unit 1) (value "U1") (footprint "Package_DIP:DIP-14_W7.62mm")
     )
     (path "/00000000-0000-0000-0000-0000625e01b4"
-      (reference "U2") (unit 1) (value "74HCT08") (footprint "Package_DIP:DIP-14_W7.62mm")
+      (reference "U2") (unit 1) (value "U2") (footprint "Package_DIP:DIP-14_W7.62mm")
     )
     (path "/00000000-0000-0000-0000-000062589459"
-      (reference "U3") (unit 1) (value "L4904") (footprint "Package_DIP:DIP-8_W7.62mm")
-    )
-  )
+      (reference "U3") (unit 1) (value "U3") (footprint "Package_DIP:DIP-8_W7.62mm")
+    )
+  )
